File: branches/PCB/Core/core_manual.brd (EAGLE design)
At the start: 51.7 x 73.7 mm, 21 parts, among them U1 PIC32MX230F064B-

Commit message: Pre Gerber for Rev 1.00
Parts:
- removed BTLDR: (no value), switch-omron:B3F-10XX
- removed PICKIT3: (no value), adafruit:1X06
- added BOOTLOADER: (no value), switch-omron:B3F-10XX
- added PICKIT1: (no value), adafruit:1X06
- moved POWER 1.80 mm to (45.7, 64.8)
- moved BARREL_JACK 1.80 mm to (7.62, 72.4)
- moved C2 1.27 mm to (21.6, 34.3)
- moved C4 1.27 mm to (39.4, 48.3)
- moved PORTB 1.27 mm to (47.0, 3.81)
- moved C3 1.27 mm to (21.6, 27.9)
- moved C5 1.27 mm to (39.4, 29.2)
- moved CRYSTAL1 1.27 mm to (14.0, 30.5)
- moved R2 1.27 mm to (2.54, 16.5)
- moved R3 1.27 mm to (24.1, 16.5)
- moved RESET 1.27 mm to (7.62, 17.8)
- moved U1 1.27 mm to (34.3, 16.5)
- moved 3V3_VREG 1.27 mm to (20.3, 55.9)
- moved C1 1.27 mm to (16.5, 47.0)
- moved PORTA 1.27 mm to (47.0, 55.9)
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Connections:
- net +3V3: now also PICKIT1.2; no longer PICKIT3.2
- net D-: now also USB_MINI_B.D-; no longer USB_MINI_B.ID
- net GND: now also BOOTLOADER.1, PICKIT1.3, USB_MINI_B.GND; no longer BTLDR.1, PICKIT3.3, USB_MINI_B.VBUS
- net MCLR: now also PICKIT1.1; no longer PICKIT3.1
- net RA0: now also PICKIT1.4; no longer PICKIT3.4
- net RA1: now also PICKIT1.5; no longer PICKIT3.5
- net RA4: now also BOOTLOADER.3; no longer BTLDR.3
- net VBUS: now also USB_MINI_B.VBUS; no longer USB_MINI_B.GND
Routing:
- net RA1: track 110.4 -> 44.0 mm
- net +3V3: track 153.1 -> 90.5 mm
- net RB0: track 59.5 -> 0.00 mm
- net RB2: track 50.4 -> 0.00 mm
- net OSC2: track 63.0 -> 13.3 mm
- net RB1: track 48.9 -> 0.00 mm
- net RA4: track 60.5 -> 17.3 mm
- net RB3: track 41.7 -> 0.00 mm
- net OSC1: track 53.5 -> 14.3 mm
- net RB4: track 33.3 -> 0.00 mm
- net D+: track 38.1 -> 65.4 mm
- net RA0: track 78.9 -> 57.5 mm
- net RB5: track 21.4 -> 0.00 mm
- net D-: track 52.1 -> 67.6 mm
- net VBUS: track 15.3 -> 7.45 mm, vias 1 -> 0
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Other:
- board size 51.7 x 73.7 mm -> 51.7 x 73.6 mm
- board text removed: "0"
- board text removed: "1"
- board text removed: "10"
- board text removed: "11"
- board text removed: "12"
- board text removed: "13"
- board text removed: "14"
- board text removed: "15"
- board text removed: "2"
- board text removed: "3"
- board text removed: "3.3V"
- board text removed: "4"
- board text removed: "5"
- board text removed: "6"
- board text removed: "7"
- board text removed: "8"
- board text removed: "9"
- board text removed: "GND"
- board text removed: "PIC32MX230F064B"
- board text removed: "VIN"
